File: MicroUK101.kicad_sch (KiCad schematic)
At the start: 31 parts, among them CON1 BARREL_JACK, J1 DB9, P1 CONN_02X02, P2 CONN_01X04, P3 CONN_02X01, P4 CONN_02X01, SW1 SW_PUSH, SW2 Switch_DPST, U1 6502, U10 74LS00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

Commit message: Release 1.02
Fix Tx and Rx lines to RS-232. Ran DRC and fixed a bunch of small track
errors. Updated silkscreen, created new gerbers.
Connections:
- net Vcc is gone; now on net VCC: U1.8 (Vcc), U5.12 (Vcc)
- net Rx: now also U4.13 (R1IN); no longer U4.8 (R2IN)
- net Tx: now also U4.14 (T1OUT); no longer U4.7 (T2OUT)
- no-connect marks 13 -> 22
Other:
- note added: "* Original Design and Schematic by Grant Searle * Mods By Steve Gray * V1.0, 2016-05-26 - Initial release. Worked but had errors * V1.01, 2022-04-26 - Fixed Power jack orientation * V1.02, 2022-05-20 - Fixed Tx and Rx line"
- note added: "32K EPROM"
- note added: "32K RAM"
- note added: "5V Centre Positive"
- note added: "ACIA"
- note added: "Board can be powered by TTL Serial Adapter"
- note added: "DRIVER"
- note added: "v1.02: fix error on original Tx and Rx connections"
- moved on the sheet: CON1, D1, P2, R4, SW2
